Commit message: +elevator controller

File: rb1_ros2_description/xacro/rb1_ros2_base.urdf.xacro (robot description, xacro)
@@ -84,10 +84,4 @@
 		<origin xyz="0.234 0.0 0.092" rpy="0 0 0"/>
 	</xacro:sensor_orbbec_astra>
-	<!-- Gazebo ros2 control plugins -->
-  <gazebo>
-    <plugin filename="libgazebo_ros2_control.so" name="gazebo_ros2_control">
-      <parameters>$(find rb1_ros2_description)/config/rb1_controller.yaml</parameters>
-    </plugin>
-  </gazebo>
 	<!-- <xacro:ros2_control/> -->
     <ros2_control name="diff_drive" type="system">
@@ -114,3 +108,24 @@
       </joint>
     </ros2_control>
+    <!-- <xacro:ros2_control/> -->
+    <ros2_control name="elevator_controller" type="system">
+      <hardware>
+          <plugin>gazebo_ros2_control/GazeboSystem</plugin>
+      </hardware>
+      <joint name="robot_elevator_platform_joint">
+        <command_interface name="effort">
+          <param name="min">0</param>
+          <param name="max">10</param>
+        </command_interface>
+        <state_interface name="position"/>
+        <state_interface name="velocity"/>
+        <state_interface name="effort"/>
+      </joint>
+    </ros2_control>
+	<!-- Gazebo ros2 control plugins -->
+  <gazebo>
+    <plugin filename="libgazebo_ros2_control.so" name="gazebo_ros2_control">
+      <parameters>$(find rb1_ros2_description)/config/rb1_controller.yaml</parameters>
+    </plugin>
+  </gazebo>
 </robot>
